File: kicad/hp3478a_fram_v2.kicad_pcb (KiCad board)
At the start: 4 copper layers, 17.8 x 29.2 mm, 18 parts, among them J1 Conn_01x11_Pin, J2 Conn_01x11_Pin, SW1 SW_DIP_x02, U1 FM16W08-SG, U2 74LVC1G58W6, U3 74LVC1G58W6, U4 74LVC1G58W6, U5 74LVC1G58W6, U6 74LVC1G58W6, U7 MCP120T-450I/TT

Commit message: fix: Voltage supervisor change (not MCP120 compatible).
Parts:
- J1, J2: value Conn_01x11_Pin -> M20-8771146
- SW1: value SW_DIP_x02 -> CHS-02TB
- U1: footprint Package_SO:SOIC-28W_7.5x17.9mm_P1.27mm -> custom_fp:SOIC-28W_7.5x17.9mm_P1.27mm
- U7: value MCP120T-450I/TT -> APX803L20-41SA; footprint Package_TO_SOT_SMD:SOT-23 -> custom_fp:SOT-23
- turned U7 to 180 degrees
Connections:
- U7 pad 1: /HP_CE2 -> GND
- U7 pad 2: +5V -> /HP_CE2
- U7 pad 3: GND -> +5V
Routing:
- net /HP_CE2: track 27.3 -> 26.0 mm
Other:
- board text added: "github.com/ mpb27/hp-3478a-fram"
- board text removed: "github.com/ mpb27/hp3478a-fram"
