File: kicad/hp3478a_fram_v2.kicad_sch (KiCad schematic)
At the start: 18 parts, among them J1 M20-8771146, J2 M20-8771146, SW1 CHS-02TB, U1 FM16W08-SG, U2 74LVC1G58W6, U3 74LVC1G58W6, U4 74LVC1G58W6, U5 74LVC1G58W6, U6 74LVC1G58W6, U7 MCP120T-450I/TT

Commit message: fix: Voltage supervisor change (not MCP120 compatible).
Parts:
- J1, J2: Manufacturer Harwin Inc. -> Harwin Inc
- U1: footprint Package_SO:SOIC-28W_7.5x17.9mm_P1.27mm -> custom_fp:SOIC-28W_7.5x17.9mm_P1.27mm
- U7: value MCP120T-450I/TT -> APX803L20-41SA; footprint Package_TO_SOT_SMD:SOT-23 -> custom_fp:SOT-23; Alternate PN APX803S-44SR-7 -> MIC803-40D3VM3; MPN MCP120T-450I/TT -> APX803S-40SR-7; Manufacturer Microchip Technology -> Diodes Inc
Connections:
- net +5V: now also U7.3 (VDD); no longer U7.2 (VDD)
- net GND: now also U7.1 (VSS); no longer U7.3 (VSS)
- net HP_CE2: now also U7.2 (~{RST}); no longer U7.1 (~{RST})
Other:
- note added: "TLV803MDBZ"
- title: (none) -> HP 3478A Calibration RAM\nFRAM Replacement
Changed lines of the file:
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@@
 	(generator_version "10.0")
 	(paper "A4")
+	(title_block
+		(title "HP 3478A Calibration RAM\\nFRAM Replacement")
+		(date "2026.09.09")
+		(rev "1")
+		(comment 1 "github.com/\\nmpb27/hp-3478a-fram")
+		(comment 2 "MB")
+		(comment 3 "MB")
+	)
+	(text "TLV803MDBZ"
+		(exclude_from_sim no)
+		(at 274.32 158.75 0)
+		(effects
+			(font
+				(size 1.27 1.27)
+			)
+		)
+	)
 	(text "FRAM_CE# <= HP_CE1# OR NOT(HP_CE2 AND NOT(HP_OD XOR HP_RW))"
 		(exclude_from_sim no)
@@
 			)
 		)
-		(property "Description" "Generic connector, single row, 01x11, script generated"
+		(property "Description" "CONN HEADER SMD 11POS 2.54MM"
 			(at 271.78 48.26 0)
 			(hide yes)
@@
 			)
 		)
-		(property "Manufacturer" "Harwin Inc."
+		(property "Manufacturer" "Harwin Inc"
 			(at 271.78 48.26 0)
 			(hide yes)
@@
 			)
 		)
-		(property "Footprint" "Package_SO:SOIC-28W_7.5x17.9mm_P1.27mm"
+		(property "Footprint" "custom_fp:SOIC-28W_7.5x17.9mm_P1.27mm"
 			(at 152.4 58.42 0)
 			(hide yes)
@@
 			)
 		)
-		(property "Description" "Generic connector, single row, 01x11, script generated"
+		(property "Description" "CONN HEADER SMD 11POS 2.54MM"
 			(at 35.56 48.26 0)
 			(hide yes)
@@
 			)
 		)
-		(property "Manufacturer" "Harwin Inc."
+		(property "Manufacturer" "Harwin Inc"
 			(at 35.56 48.26 0)
 			(hide yes)
@@
 			)
 		)
-		(property "Description" "2x DIP Switch, Single Pole Single Throw (SPST) switch, small symbol"
+		(property "Description" "SWITCH SLIDE DIP SPST 0.1A 6V"
 			(at 81.28 63.5 0)
 			(hide yes)
@@
 		(in_pos_files yes)
 		(dnp no)
-		(fields_autoplaced yes)
 		(property "Reference" "U7"
 			(at 267.97 151.1299 0)
@@
 			)
 		)
-		(property "Value" "MCP120T-450I/TT"
+		(property "Value" "APX803L20-41SA"
 			(at 267.97 153.6699 0)
 			(show_name no)
@@
 			)
 		)
-		(property "Footprint" "Package_TO_SOT_SMD:SOT-23"
+		(property "Footprint" "custom_fp:SOT-23"
 			(at 246.38 161.29 0)
 			(hide yes)
@@
 			)
 		)
-		(property "Description" "IC SUPERVISOR 1CH 4.50V SOT-23"
+		(property "Description" "IC SUPERVISOR 1CH 4.0V SOT-23"
 			(at 261.62 152.4 0)
 			(hide yes)
@@
 			)
 		)
-		(property "Alternate PN" "APX803S-44SR-7"
-			(at 261.62 152.4 0)
-			(hide yes)
+		(property "Alternate PN" "MIC803-40D3VM3"
+			(at 276.86 156.21 0)
 			(show_name no)
 			(do_not_autoplace no)
@@
 			)
 		)
-		(property "MPN" "MCP120T-450I/TT"
+		(property "MPN" "APX803S-40SR-7"
 			(at 261.62 152.4 0)
 			(hide yes)
@@
 			)
 		)
-		(property "Manufacturer" "Microchip Technology"
+		(property "Manufacturer" "Diodes Inc"
 			(at 261.62 152.4 0)
 			(hide yes)

Commit message: fix: Fixed part number for U7 voltage supervisor.
Parts:
- U7: MPN APX803S-40SR-7 -> APX803L20-41SA
Changed lines of the file:
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@@
 			)
 		)
-		(property "MPN" "APX803S-40SR-7"
+		(property "MPN" "APX803L20-41SA"
 			(at 261.62 152.4 0)
 			(hide yes)
